File: Hardware/back/back.kicad_sch (KiCad schematic)
At the start: 2 parts, among them J1 Conn_01x06_Male

Commit message: Major HW and FW improvements
Parts:
- removed BT1: Battery_Cell, Battery:BatteryHolder_Keystone_103_1x20mm, symbol Device:Battery_Cell
- removed J1: Conn_01x06_Male, Connector_PinHeader_2.54mm:PinHeader_2x03_P2.54mm_Vertical_SMD, symbol Connector:Conn_01x06_Male
Connections:
- no-connect marks 4 -> 0
Changed lines of the file:
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@@
-(kicad_sch (version 20211123) (generator eeschema)
-  (paper "A4")
-  (no_connect (at 158.75 92.71))
-  (no_connect (at 158.75 95.25))
-  (no_connect (at 158.75 97.79))
-  (no_connect (at 158.75 102.87))
-  (wire (pts (xy 148.59 100.33) (xy 158.75 100.33))
-    (stroke (width 0) (type default) (color 0 0 0 0))
-  )
-  (wire (pts (xy 148.59 90.17) (xy 158.75 90.17))
-    (stroke (width 0) (type default) (color 0 0 0 0))
-  )
-  (wire (pts (xy 148.59 92.71) (xy 148.59 90.17))
-    (stroke (width 0) (type default) (color 0 0 0 0))
-  )
-  (symbol (lib_id "Device:Battery_Cell") (at 148.59 97.79 0) (unit 1)
-    (in_bom yes) (on_board yes)
-    (property "Reference" "BT1" (id 0) (at 151.5872 95.3516 0)
-      (effects (font (size 1.27 1.27)) (justify left))
-    )
-    (property "Value" "Battery_Cell" (id 1) (at 151.5872 97.663 0)
-      (effects (font (size 1.27 1.27)) (justify left))
-    )
-    (property "Footprint" "Battery:BatteryHolder_Keystone_103_1x20mm" (id 2) (at 148.59 96.266 90)
-      (effects (font (size 1.27 1.27)) hide)
-    )
-    (property "Datasheet" "~" (id 3) (at 148.59 96.266 90)
-      (effects (font (size 1.27 1.27)) hide)
-    )
-    (pin "1")
-    (pin "2")
-  )
-  (symbol (lib_id "Connector:Conn_01x06_Male") (at 163.83 95.25 0) (mirror y) (unit 1)
-    (in_bom yes) (on_board yes)
-    (property "Reference" "J1" (id 0) (at 164.5412 95.9104 0)
-      (effects (font (size 1.27 1.27)) (justify right))
-    )
-    (property "Value" "Conn_01x06_Male" (id 1) (at 164.5412 98.2218 0)
-      (effects (font (size 1.27 1.27)) (justify right))
-    )
-    (property "Footprint" "Connector_PinHeader_2.54mm:PinHeader_2x03_P2.54mm_Vertical_SMD" (id 2) (at 163.83 95.25 0)
-      (effects (font (size 1.27 1.27)) hide)
-    )
-    (property "Datasheet" "~" (id 3) (at 163.83 95.25 0)
-      (effects (font (size 1.27 1.27)) hide)
-    )
-    (pin "1")
-    (pin "2")
-    (pin "3")
-    (pin "4")
-    (pin "5")
-    (pin "6")
-  )
-  (sheet_instances
-    (path "/" (page "1"))
-  )
-  (symbol_instances
-    (path "/00000000-0000-0000-0000-00005eff28d6"
-      (reference "BT1") (unit 1) (value "Battery_Cell") (footprint "Battery:BatteryHolder_Keystone_103_1x20mm")
-    )
-    (path "/00000000-0000-0000-0000-00005eff3181"
-      (reference "J1") (unit 1) (value "Conn_01x06_Male") (footprint "Connector_PinHeader_2.54mm:PinHeader_2x03_P2.54mm_Vertical_SMD")
-    )
-  )
+(kicad_sch
+	(version 20231120)
+	(generator "eeschema")
+	(generator_version "8.0")
+	(paper "A4")
+	(sheet_instances
+		(path "/"
+			(page "1")
+		)
+	)
 )
