File: Hardware/mcu board/mcu board.kicad_pcb (KiCad board)
At the start: 2 copper layers, 103 x 90 mm, 50 parts, among them J1 Conn_01x10_Male, J2 Conn_01x06_Male, J3 Conn_01x06_Male, J4 Conn_01x06_Male, J5 USB_C_Receptacle_USB2.0, J6 Conn_01x06_Male, Q1 NMOS, SW1 SW_Push, U1 AP1117-33, U2 STM32F103C8Tx, U3 MIC4427, U4 ICL7660, Y1 8MHz, Y2 32.768k

Commit message: Major HW and FW improvements
Parts:
- removed J2, J3, J6: Conn_01x06_Male, Connector_PinHeader_2.54mm:PinHeader_2x03_P2.54mm_Vertical_SMD
- removed R3: 0R, Resistor_SMD:R_1206_3216Metric_Pad1.30x1.75mm_HandSolder
- added BT1: Battery_Cell, Battery:BatteryHolder_Seiko_MS621F, F.Cu at (134.8, 89.5)
- added C18: CGA0603X5R105K160JT, Capacitor_SMD:C_0603_1608Metric_Pad1.08x0.95mm_HandSolder, F.Cu at (104.0, 138.9)
- added C19: CGA0603X5R105K160JT, Capacitor_SMD:C_0603_1608Metric_Pad1.08x0.95mm_HandSolder, F.Cu at (127.8, 139.1)
- added C20: CGA0603X5R105K160JT, Capacitor_SMD:C_0603_1608Metric_Pad1.08x0.95mm_HandSolder, F.Cu at (157.0, 139.2)
- added C21: CGA0603X5R105K160JT, Capacitor_SMD:C_0603_1608Metric_Pad1.08x0.95mm_HandSolder, F.Cu at (179.9, 139.0)
- added D10: 1N5819, Diode_SMD:D_SOD-123, F.Cu at (133.1, 84.3)
- added D11: 1N5819, Diode_SMD:D_SOD-123, F.Cu at (132.0, 86.6)
- added D4: SMAJ5.0A, Diode_SMD:D_SMA, F.Cu at (138.5, 80.0)
- added D5: SMAJ250A, Diode_SMD:D_SMA, F.Cu at (170.3, 80.9)
- added D6: WS2812B, LED_SMD:LED_WS2812B_PLCC4_5.0x5.0mm_P3.2mm, F.Cu at (108.7, 138.9)
- added D7: WS2812B, LED_SMD:LED_WS2812B_PLCC4_5.0x5.0mm_P3.2mm, F.Cu at (132.2, 138.9)
- added D8: WS2812B, LED_SMD:LED_WS2812B_PLCC4_5.0x5.0mm_P3.2mm, F.Cu at (161.4, 138.9)
- added D9: WS2812B, LED_SMD:LED_WS2812B_PLCC4_5.0x5.0mm_P3.2mm, F.Cu at (184.4, 138.9)
- added J7: HCZZ0015-5, Connector_Molex:Molex_PicoBlade_53398-0571_1x05-1MP_P1.25mm_Vertical, F.Cu at (137.6, 115.5)
- added J8: HCZZ0015-5, Connector_Molex:Molex_PicoBlade_53398-0571_1x05-1MP_P1.25mm_Vertical, F.Cu at (163.5, 80.5)
- added R11: 5k1, Resistor_SMD:R_0402_1005Metric_Pad0.72x0.64mm_HandSolder, F.Cu at (134.9, 86.6)
- added SW2: XKB5858-W-F-75, nixie:XKB5858-W-F-75, F.Cu at (130.6, 63.5)
- added SW3: XKB5858-W-F-75, nixie:XKB5858-W-F-75, F.Cu at (141.6, 63.5)
- added SW4: XKB5858-W-F-75, nixie:XKB5858-W-F-75, F.Cu at (152.6, 63.5)
- added SYM1: SYM_Flash_Large, custom:HighVoltage, F.Cu at (151.7, 76.6)
- C1, C2, C3, C4: footprint Capacitor_SMD:C_1206_3216Metric_Pad1.33x1.80mm_HandSolder -> Capacitor_SMD:C_0402_1005Metric_Pad0.74x0.62mm_HandSolder
- C10, C11, C5, C6, C7, C8, C9: value 1uF -> CGA0603X5R105K160JT; footprint Capacitor_SMD:C_1206_3216Metric_Pad1.33x1.80mm_HandSolder -> Capacitor_SMD:C_0603_1608Metric_Pad1.08x0.95mm_HandSolder
- C12, C13: value 4.7uF -> 189RV165
- C17: value 220uF -> GVE1C477M0810CNVC
- D1: footprint Diode_SMD:D_SMA_Handsoldering -> Diode_SMD:D_SMA
- D2, D3: footprint Diode_SMD:D_SOD-323_HandSoldering -> Diode_SMD:D_SOD-123
- F1: value Polyfuse -> JK-MSMD050-30
- H1, H2, H3, H4: value MountingHole -> SMTSO3080MTJ; footprint MountingHole:MountingHole_3.2mm_M3 -> Mounting_Wuerth:Mounting_Wuerth_WA-SMSI-M3_H8mm_9774080360
- J1: value Conn_01x10_Male -> HCZZ0015-5; footprint Connector_PinHeader_2.54mm:PinHeader_2x05_P2.54mm_Vertical_SMD -> Connector_Molex:Molex_PicoBlade_53398-0571_1x05-1MP_P1.25mm_Vertical
- J4: value Conn_01x06_Male -> HCZZ0015-5; footprint Connector_PinHeader_2.54mm:PinHeader_2x03_P2.54mm_Vertical_SMD -> Connector_Molex:Molex_PicoBlade_53398-0571_1x05-1MP_P1.25mm_Vertical
- L1: value 220uH -> CYH127-220UH
- Q1: value NMOS -> STD4NK60ZT4
- R1, R2, R7: value 10k -> 5k1; footprint Resistor_SMD:R_1206_3216Metric_Pad1.30x1.75mm_HandSolder -> Resistor_SMD:R_0402_1005Metric_Pad0.72x0.64mm_HandSolder
- R10: value 0R -> 10R; footprint Resistor_SMD:R_1206_3216Metric_Pad1.30x1.75mm_HandSolder -> Resistor_SMD:R_0402_1005Metric_Pad0.72x0.64mm_HandSolder
- R4, R5, R6: footprint Resistor_SMD:R_1206_3216Metric_Pad1.30x1.75mm_HandSolder -> Resistor_SMD:R_0402_1005Metric_Pad0.72x0.64mm_HandSolder
- R9: value NC -> 10R; footprint Resistor_SMD:R_1206_3216Metric_Pad1.30x1.75mm_HandSolder -> Resistor_SMD:R_0402_1005Metric_Pad0.72x0.64mm_HandSolder
- SW1: value SW_Push -> TS-1101-C-W; footprint Button_Switch_SMD:SW_Push_1P1T_NO_6x6mm_H9.5mm -> Button_Switch_SMD:SW_SPST_CK_RS282G05A3
- U3: value MIC4427 -> NSG4427
- U4: value ICL7660 -> TC7660M/TR
- Y1: value 8MHz -> TAXM8M4RFDCET2T; footprint Crystal:Crystal_SMD_HC49-SD -> Crystal:Crystal_SMD_3225-4Pin_3.2x2.5mm
- Y2: value 32.768k -> XKXGI-SUA-32.768K
- moved R2 16.2 mm to (129.0, 103.8)
- moved C2 9.75 mm to (121.0, 93.8), turned to 0 degrees
- moved Q1 6.78 mm to (170.1, 109.8)
- moved C4 6.56 mm to (125.3, 97.6)
- moved C1 5.88 mm to (123.3, 96.7)
- moved R7 5.48 mm to (163.9, 109.9)
- moved R10 5.31 mm to (149.9, 102.2), turned to 180 degrees
- moved F1 5.11 mm to (127.4, 70.1)
- moved C3 4.64 mm to (125.3, 95.4), turned to -90 degrees
- moved J1 4.29 mm to (137.6, 109.6), turned to 0 degrees
- moved SW1 4.27 mm to (113.7, 96.0), turned to 180 degrees
- moved Y1 4.09 mm to (121.0, 96.5)
- moved J4 3.90 mm to (148.6, 94.8), turned to 90 degrees
- moved C5 3.40 mm to (109.8, 83.9), turned to 0 degrees
- moved H1 3.35 mm to (106.0, 69.5)
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Connections:
- C1 pad 1: Net-(C1-Pad1) -> Net-(U2-PD0)
- C2 pad 1: Net-(C2-Pad1) -> Net-(U2-PD1)
- J1 pad 1: /PA4 -> /PA5
- J1 pad 2: /PA5 -> /PA7
- J1 pad 3: /PA6 -> /PB1
- J1 pad 4: /PA7 -> /PB10
- J1 pad 5: Net-(J1-Pad5) -> +5V
- J4 pad 1: Net-(J4-Pad1) -> Net-(J4-Pin_1)
- J4 pad 2: Net-(J4-Pad2) -> Net-(J4-Pin_2)
- J4 pad 3: Net-(J4-Pad3) -> +3V3
- J4 pad 5: +3V3 -> GND
- R1 pad 1: GND -> Net-(U2-BOOT0)
- R1 pad 2: Net-(R1-Pad2) -> GND
- R10 pad 2: Net-(J4-Pad1) -> Net-(U2-PA9)
- R2 pad 1: Net-(R2-Pad1) -> +3V3
- R2 pad 2: +3V3 -> Net-(U2-NRST)
- SW1 pad 1: Net-(R2-Pad1) -> Net-(U2-NRST)
- U2 pad 10: Net-(J3-Pad1) -> /PA0
- U2 pad 11: Net-(J3-Pad2) -> /PA1
- U2 pad 12: unconnected-(U2-Pad12) -> /PA2
- U2 pad 13: unconnected-(U2-Pad13) -> /PA3
- U2 pad 18: Net-(J1-Pad5) -> /PB0
- U2 pad 19: Net-(J1-Pad6) -> /PB1
- U2 pad 20: Net-(J1-Pad7) -> /PB2
- U2 pad 21: Net-(J1-Pad8) -> /PB10
- U2 pad 22: unconnected-(U2-Pad22) -> /PB11
- U2 pad 30: Net-(J4-Pad1) -> Net-(U2-PA9)
- U2 pad 31: Net-(J4-Pad2) -> Net-(J4-Pin_1)
- U2 pad 34: Net-(J4-Pad3) -> Net-(J4-Pin_2)
- U2 pad 44: Net-(R1-Pad2) -> Net-(U2-BOOT0)
- U2 pad 5: Net-(C1-Pad1) -> Net-(U2-PD0)
- U2 pad 6: Net-(C2-Pad1) -> Net-(U2-PD1)
- U2 pad 7: Net-(R2-Pad1) -> Net-(U2-NRST)
- Y1 pad 1: Net-(C1-Pad1) -> Net-(U2-PD1)
- Y1 pad 2: Net-(C2-Pad1) -> GND
Routing:
- net +5V: track 134.7 -> 263.2 mm
- net /PA2: track 0.00 -> 110.4 mm
- net /PA1: track 0.00 -> 98.0 mm
- net /PA0: track 0.00 -> 85.8 mm
- net /PA3: track 0.00 -> 49.4 mm
- net Net-(R2-Pad1): track 35.8 -> 0.00 mm
- net Net-(D7-DOUT): track 0.00 -> 35.5 mm
- net GND: track 122.8 -> 92.1 mm
- net +3V3: track 112.4 -> 82.5 mm
- net Net-(D6-DOUT): track 0.00 -> 29.8 mm
- net Net-(D8-DOUT): track 0.00 -> 29.3 mm
- net Net-(J3-Pad2): track 27.3 -> 0.00 mm
- net Net-(J4-Pad1): track 23.7 -> 0.00 mm
- net Net-(U2-NRST): track 0.00 -> 22.4 mm
- net Net-(J3-Pad1): track 20.1 -> 0.00 mm
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- removed copper zone on F.Cu, net Net-(D1-A)
Other:
- board size 103 x 90 mm -> 100 x 90 mm
- rule pad_to_mask_clearance: 0.051 -> 0
- board text added: "Designed by K.K."
- board text added: "⎓250 V"
- board text removed: "Designed by Kononenko K."
