File: Hardware/mcu board/mcu board.kicad_sch (KiCad schematic)
At the start: 50 parts, among them J1 Conn_01x10_Male, J2 Conn_01x06_Male, J3 Conn_01x06_Male, J4 Conn_01x06_Male, J5 USB_C_Receptacle_USB2.0, J6 Conn_01x06_Male, Q1 STD4NK60ZT4, SW1 SW_Push, U1 AP1117-33, U2 STM32F103C8Tx, U3 MIC4427, U4 ICL7660, Y1 8MHz, Y2 32.768k

Commit message: Major HW and FW improvements
Parts:
- removed H1, H2, H3, H4: MountingHole, MountingHole:MountingHole_3.2mm_M3, symbol Mechanical:MountingHole
- removed J1: Conn_01x10_Male, Connector_PinHeader_2.54mm:PinHeader_2x05_P2.54mm_Vertical_SMD, symbol Connector:Conn_01x10_Male
- removed J2, J3, J4, J6: Conn_01x06_Male, Connector_PinHeader_2.54mm:PinHeader_2x03_P2.54mm_Vertical_SMD, symbol Connector:Conn_01x06_Male
- removed R3: 0R, Resistor_SMD:R_1206_3216Metric_Pad1.30x1.75mm_HandSolder, symbol Device:R
- removed Y1: 8MHz, Crystal:Crystal_SMD_HC49-SD, symbol Device:Crystal
- added BT1: Battery_Cell, Battery:BatteryHolder_Seiko_MS621F, symbol Device:Battery_Cell
- added C18, C19, C20, C21: CGA0603X5R105K160JT, Capacitor_SMD:C_0603_1608Metric_Pad1.08x0.95mm_HandSolder, symbol Device:C
- added D10, D11: 1N5819, Diode_SMD:D_SOD-123, symbol Device:D
- added D4: SMAJ5.0A, Diode_SMD:D_SMA, symbol Diode:SMAJ5.0A
- added D5: SMAJ250A, Diode_SMD:D_SMA, symbol Diode:SMAJ250A
- added D6, D7, D8, D9: WS2812B, LED_SMD:LED_WS2812B_PLCC4_5.0x5.0mm_P3.2mm, symbol LED:WS2812B
- added H1, H2, H3, H4: SMTSO3080MTJ, Mounting_Wuerth:Mounting_Wuerth_WA-SMSI-M3_H8mm_9774080360, symbol Mechanical:MountingHole_Pad
- added J1, J4, J7, J8: HCZZ0015-5, Connector_Molex:Molex_PicoBlade_53398-0571_1x05-1MP_P1.25mm_Vertical, symbol Connector_Generic_MountingPin:Conn_01x05_MountingPin
- added R11: 5k1, Resistor_SMD:R_0402_1005Metric_Pad0.72x0.64mm_HandSolder, symbol Device:R
- added SW2, SW3, SW4: XKB5858-W-F-75, nixie:XKB5858-W-F-75, symbol Switch:SW_Push
- added SYM1: SYM_Flash_Large, custom:HighVoltage, symbol Graphic:SYM_Flash_Large
- added Y1: TAXM8M4RFDCET2T, Crystal:Crystal_SMD_3225-4Pin_3.2x2.5mm, symbol Device:Crystal_GND24
- C1, C2, C3, C4: footprint Capacitor_SMD:C_1206_3216Metric_Pad1.33x1.80mm_HandSolder -> Capacitor_SMD:C_0402_1005Metric_Pad0.74x0.62mm_HandSolder; Manufacturer (none) -> YAGEO; Part Number (none) -> CC0402JRNPO9BN180
- C10, C11, C5, C6, C7, C8, C9: value 1uF -> CGA0603X5R105K160JT; footprint Capacitor_SMD:C_1206_3216Metric_Pad1.33x1.80mm_HandSolder -> Capacitor_SMD:C_0603_1608Metric_Pad1.08x0.95mm_HandSolder; Manufacturer (none) -> YAGEO; Part Number (none) -> CC0603KRX5R8BB105
- C12, C13: value 4.7uF -> 189RV165; Manufacturer (none) -> KNSCHA; Part Number (none) -> 189RV165
- C14, C15, C16: Manufacturer (none) -> YAGEO; Part Number (none) -> CC1206KKX5R8BB106
- C17: value 220uF -> GVE1C477M0810CNVC; Manufacturer (none) -> HRK; Part Number (none) -> GVE1C477M0810CNVC
- D1: footprint Diode_SMD:D_SMA_Handsoldering -> Diode_SMD:D_SMA; Manufacturer (none) -> JSMSEMI; Part Number (none) -> US1M
- D2, D3: footprint Diode_SMD:D_SOD-323_HandSoldering -> Diode_SMD:D_SOD-123; Manufacturer (none) -> Diodes Incorporated; Part Number (none) -> 1N5819HW-7-F
- F1: value Polyfuse -> JK-MSMD050-30; Manufacturer (none) -> Jinrui Electronic Materials Co.; Part Number (none) -> JK-MSMD050-30
- J5: Manufacturer (none) -> Korean Hroparts Elec; Part Number (none) -> TYPE-C-31-M-12
- L1: value 220uH -> CYH127-220UH; Manufacturer (none) -> SHOU HAN CYH125-330UH; Part Number (none) -> SHOU HAN CYH125-330UH
- Q1: Manufacturer (none) -> STMicroelectronics; Part Number (none) -> STD4NK60ZT4
- R1, R2, R7: value 10k -> 5k1; footprint Resistor_SMD:R_1206_3216Metric_Pad1.30x1.75mm_HandSolder -> Resistor_SMD:R_0402_1005Metric_Pad0.72x0.64mm_HandSolder; Manufacturer (none) -> YAGEO; Part Number (none) -> RC0402FR-075K1L
- R10: value 0R -> 10R; footprint Resistor_SMD:R_1206_3216Metric_Pad1.30x1.75mm_HandSolder -> Resistor_SMD:R_0402_1005Metric_Pad0.72x0.64mm_HandSolder; Manufacturer (none) -> YAGEO; Part Number (none) -> RC0402FR-0710RL
- R4, R5: footprint Resistor_SMD:R_1206_3216Metric_Pad1.30x1.75mm_HandSolder -> Resistor_SMD:R_0402_1005Metric_Pad0.72x0.64mm_HandSolder; Manufacturer (none) -> YAGEO; Part Number (none) -> RC0402FR-075K1L
- R6: footprint Resistor_SMD:R_1206_3216Metric_Pad1.30x1.75mm_HandSolder -> Resistor_SMD:R_0402_1005Metric_Pad0.72x0.64mm_HandSolder; Manufacturer (none) -> YAGEO; Part Number (none) -> RC0402FR-0710RL
- R8: Manufacturer (none) -> YAGEO; Part Number (none) -> RC1206FR-071ML
- R9: value NC -> 10R; footprint Resistor_SMD:R_1206_3216Metric_Pad1.30x1.75mm_HandSolder -> Resistor_SMD:R_0402_1005Metric_Pad0.72x0.64mm_HandSolder; now not fitted
- SW1: value SW_Push -> TS-1101-C-W; footprint Button_Switch_SMD:SW_Push_1P1T_NO_6x6mm_H9.5mm -> Button_Switch_SMD:SW_SPST_CK_RS282G05A3; now not fitted
- U1: Manufacturer (none) -> UMW(Youtai Semiconductor Co., Ltd.); Part Number (none) -> AMS1117-3.3
- U2: Manufacturer (none) -> STMicroelectronics; Part Number (none) -> STM32F103C8T6
- U3: value MIC4427 -> NSG4427; Manufacturer (none) -> WXNSIC; Part Number (none) -> NSG4427
- U4: value ICL7660 -> TC7660M/TR; Manufacturer (none) -> HGSEMI; Part Number (none) -> TC7660M/TR
- Y2: value 32.768k -> XKXGI-SUA-32.768K; Manufacturer (none) -> YXC Crystal Oscillators; Part Number (none) -> XKXGI-SUA-32.768K
Connections:
- net +3V3: now also R2.1, D10.2 (A), J4.3 (Pin_3); no longer R2.2
- net +5V: now also C18.2, C19.2, C20.2, C21.2, D4.1 (A1), D6.1 (VDD), D7.1 (VDD), D8.1 (VDD), D9.1 (VDD), J1.5 (Pin_5)
- net GND: now also R1.2, BT1.2 (-), C18.1, C19.1, C20.1, C21.1, D4.2 (A2), D5.2 (A2), D6.3 (VSS), D7.3 (VSS), D8.3 (VSS), D9.3 (VSS), H1.1, H2.1, H3.1, H4.1, J1.MP (MountPin), J4.5 (Pin_5), J4.MP (MountPin), J7.5 (Pin_5), J7.MP (MountPin), J8.5 (Pin_5), SW2.2, SW3.2, SW4.2, Y1.2, Y1.4; no longer R1.1
- net PA4: now also J7.1 (Pin_1)
- net PA5: now also J1.1 (Pin_1)
- net PA6: now also J7.2 (Pin_2)
- net PA7: now also J1.2 (Pin_2)
- net at C7.2, U2.1 (VBAT): now also D11.1 (K)
- net PA0: now reaches U2.10 (PA0)
- net PA0: now also SW2.1
- net PA1: now reaches U2.11 (PA1)
- net PA1: now also SW3.1
- net PA2: now reaches U2.12 (PA2)
- net PA2: now also SW4.1
- net PA3: now reaches U2.13 (PA3)
- net PA3: now also D6.4 (DIN)
- net PB0: now reaches U2.18 (PB0)
- net PB0: now also J7.3 (Pin_3)
- net PB1: now reaches U2.19 (PB1)
- net PB1: now also J1.3 (Pin_3)
- net PB2: now reaches U2.20 (PB2)
- net PB2: now also J7.4 (Pin_4)
- net PB10: now reaches U2.21 (PB10)
- net PB10: now also J1.4 (Pin_4)
- net PB11: now reaches U2.22 (PB11)
- net at U2.31 (PA10): now also J4.1 (Pin_1)
- net at U2.34 (PA13): now also J4.2 (Pin_2)
- net at U2.37 (PA14): now also J4.4 (Pin_4)
- net at U2.44 (BOOT0): now also R1.1; no longer R1.2
- net at C1.1, U2.5 (PD0): now also Y1.3
- net at C2.1, U2.6 (PD1): now also Y1.1
- net at SW1.1, U2.7 (NRST): now also R2.2; no longer R2.1
- net at C12.1, C13.1, D1.1 (K)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: now also D5.1 (A1), J8.1 (Pin_1)
- new net: D8.2 (DOUT), D9.4 (DIN)
- new net: D7.2 (DOUT), D8.4 (DIN)
- new net: BT1.1 (+), D11.2 (A), R11.2
- new net: D6.2 (DOUT), D7.4 (DIN)
- new net: D10.1 (K), R11.1
- no-connect marks 33 -> 31
Other:
- moved on the sheet: C1, C10, C11, C17, C2, C3, C4, C5, C6, C8, C9, U1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
