File: Hardware/nixie display/nixie display.kicad_sch (KiCad schematic)
At the start: 36 parts, among them J1 Conn_01x05_Male, J2 Conn_01x03_Male, J3 Conn_01x02_Male, J4 Conn_01x02_Male, J5 Conn_01x05_Male, J6 Conn_01x02_Male, Q1 MJE13003, Q2 Q_NMOS_GSD, U1 K155ID1, U10 TLP627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

Commit message: Major HW and FW improvements
Parts:
- removed BZ1: Buzzer, Buzzer_Beeper:Buzzer_12x9.5RM7.6, symbol Device:Buzzer
- removed D1: SS14, Diode_SMD:D_SMA_Handsoldering, symbol Device:D_Schottky
- removed J1, J5: Conn_01x05_Male, Connector_PinHeader_2.54mm:PinHeader_1x05_P2.54mm_Vertical, symbol Connector:Conn_01x05_Male
- removed J2: Conn_01x03_Male, Connector_PinHeader_2.54mm:PinHeader_1x03_P2.54mm_Vertical, symbol Connector:Conn_01x03_Male
- removed J3: Conn_01x02_Male, Connector_PinHeader_2.54mm:PinHeader_1x02_P2.54mm_Vertical, symbol Connector:Conn_01x02_Male
- removed J4, J6: Conn_01x02_Male, nixie clock:PinHeader_1x02_P5.08mm_Vertical, symbol Connector:Conn_01x02_Male
- removed Q2: Q_NMOS_GSD, Package_TO_SOT_SMD:SOT-23, symbol Device:Q_NMOS_GSD
- removed R11, R7: 100, Resistor_SMD:R_1206_3216Metric_Pad1.42x1.75mm_HandSolder, symbol Device:R
- removed R12, R8: 10k, Resistor_SMD:R_1206_3216Metric_Pad1.42x1.75mm_HandSolder, symbol Device:R
- added J1, J2, J3, J5: HCZZ0015-5, Connector_Molex:Molex_PicoBlade_53398-0571_1x05-1MP_P1.25mm_Vertical, symbol Connector_Generic_MountingPin:Conn_01x05_MountingPin
- added R1: 47k, Resistor_SMD:R_1206_3216Metric_Pad1.30x1.75mm_HandSolder, symbol Device:R
- added R2: 100, Resistor_SMD:R_1206_3216Metric_Pad1.30x1.75mm_HandSolder, symbol Device:R
- added SYM1: SYM_Flash_Large, custom:HighVoltage, symbol Graphic:SYM_Flash_Large
- C1: Manufacturer (none) -> YAGEO; Part Number (none) -> CC1206KKX7R9BB105
- DS1, DS2, DS3, DS4: Part Number (none) -> IN12
- NE1, NE2: Part Number (none) -> NE-2
- Q1: value MJE13003 -> FJT44; footprint Package_TO_SOT_THT:TO-126-3_Vertical -> Package_TO_SOT_SMD:SOT-223-3_TabPin2; Manufacturer (none) -> WEIDA; Part Number (none) -> FJT44
- R10, R9: value 100k -> 47k; Manufacturer (none) -> YAGEO; Part Number (none) -> RC1206JR-0747KL
- R13, R14, R15, R16: Manufacturer (none) -> YAGEO; Part Number (none) -> RC1206JR-0747KL
- R17, R18, R19, R20: Manufacturer (none) -> YAGEO; Part Number (none) -> RC1206JR-07100RL
- U1: value K155ID1 -> DS1009-16AT1NX-0A2; Manufacturer (none) -> CONNFLY Elec; Part Number (none) -> DS1009-16AT1NX-0A2
- U10, U7, U8, U9: Manufacturer (none) -> TOSHIBA; Part Number (none) -> TLP627(TP1,F)
Connections:
- net +5V: now also J3.1 (Pin_1)
- net A1: now also J1.1 (Pin_1)
- net A2: now also J1.2 (Pin_2)
- net A3: now also J1.3 (Pin_3)
- net A4: now also J1.4 (Pin_4)
- net D0: now also J2.1 (Pin_1)
- net D1: now also J2.3 (Pin_3)
- net D2: now also J2.4 (Pin_4)
- net D3: now also J2.2 (Pin_2)
- net GND: now also J1.5 (Pin_5), J2.5 (Pin_5), J3.4 (Pin_4), J3.5 (Pin_5), J5.5 (Pin_5), R1.1
- net VCC: now also J5.1 (Pin_1)
- net at Q1.1 (B): now also R1.2, R2.2
- new net: J3.3 (Pin_3), R2.1
- no-connect marks 0 -> 8
